File: scoppy/scoppy_control.kicad_pcb (KiCad board)
At the start: 2 copper layers, 30.4 x 100 mm, 39 parts, among them J1 CH1, J2 CH2, J4 CH1_Through, J5 CH2_Through, J8 USB_A, SW1 AC/DCcoupling, SW2 AC/DCcoupling, SW3 Switch±30V/±8V/, SW4 Switch±30V/±8V/

Commit message: AddFile
Parts:
- moved SW3 19.1 mm to (107.5, 81.4)
- moved SW4 19.1 mm to (126.9, 81.4)
- moved C10 12.0 mm to (127.0, 73.2), turned to -90 degrees
- moved R8 10.6 mm to (132.8, 75.8)
- moved R12 9.63 mm to (116.7, 90.1)
- moved C15 9.40 mm to (106.5, 76.3), turned to 0 degrees
- moved C5 9.20 mm to (112.9, 68.0)
- moved C6 9.20 mm to (133.1, 68.0)
- moved R17 8.85 mm to (111.7, 62.3)
- moved R18 8.34 mm to (125.1, 62.8)
- moved C9 6.76 mm to (118.3, 82.8)
- moved R7 6.43 mm to (113.6, 76.4), turned to 90 degrees
Routing:
- net GND: track 149.0 -> 128.6 mm
- net GPIO5: track 65.9 -> 46.6 mm
- net GPIO4: track 69.5 -> 50.4 mm
- net Net-(R15-Pad2): track 12.1 -> 30.7 mm
- net Net-(R18-Pad2): track 7.19 -> 24.7 mm
- net GPIO3: track 75.9 -> 60.3 mm
- net Net-(R17-Pad2): track 9.56 -> 23.6 mm
- net Net-(R16-Pad2): track 7.44 -> 19.3 mm
- net Net-(C4-Pad2): track 43.5 -> 54.2 mm
- net GPIO2: track 70.0 -> 60.1 mm
- net Net-(C3-Pad2): track 43.3 -> 52.6 mm
- net -3V3: track 93.7 -> 102.9 mm
- net Net-(C12-Pad1): track 76.0 -> 85.0 mm
- net Net-(C13-Pad1): track 102.4 -> 107.3 mm
- net Net-(C19-Pad2): track 41.9 -> 38.2 mm
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