File: scoppy/scoppy_panel.kicad_pcb (KiCad board)
At the start: 2 copper layers, 30.4 x 128.5 mm, 11 parts

Commit message: AddFile
Parts:
- removed REF10, REF11: MountingHole_3.2mm_M3, MountingHole:MountingHole_3.2mm_M3
- added REF12: MountingHole_3.2mm_M3_DIN965_Pad, MountingHole:MountingHole_3.2mm_M3_DIN965_Pad, F.Cu at (178.0, 153.0)
- added REF12: MountingHole_3.2mm_M3_DIN965_Pad, MountingHole:MountingHole_3.2mm_M3_DIN965_Pad, F.Cu at (162.6, 30.5)
- moved REF1 19.1 mm to (160.6, 65.5)
- moved REF2 19.1 mm to (180.0, 65.5)
Routing:
- added copper zone on B.Cu, net GND
- added copper zone on F.Cu, net GND
Other:
- board text added: "ijnekenamay"
- board text added: "jlcjlcjlcjlc"
